File: PCB/Keyboard.kicad_pcb (KiCad board)
At the start: 2 copper layers, 28 x 18 mm, 25 parts, among them P1 USB_OTG, SW1 RST, U1 ATMEGA32U4-QFN44, X1 ABM10-16.000MHZ-D30-T3

Commit message: Mad junk I was trying in the past
Parts:
- removed ISP1: ATMEL_ISP-6P, SMD-Connectors:ISP-PADS_2mm54
- added J1: RESET, RB-SMD-Connectors:TESTPOINT-1mm-NO_TEXT, B.Cu at (151.0, 110.0)
- added J2: SCK, RB-SMD-Connectors:TESTPOINT-1mm-NO_TEXT, B.Cu at (151.0, 112.0)
- added J3: MISO, RB-SMD-Connectors:TESTPOINT-1mm-NO_TEXT, B.Cu at (151.0, 114.0)
- added J4: MOSI, RB-SMD-Connectors:TESTPOINT-1mm-NO_TEXT, B.Cu at (153.0, 114.0)
- added J5: VBUS, RB-SMD-Connectors:TESTPOINT-1mm-NO_TEXT, B.Cu at (156.0, 101.0)
- added J6: 5V, RB-SMD-Connectors:TESTPOINT-1mm-NO_TEXT, B.Cu at (153.0, 112.0)
- added J7: D-, RB-SMD-Connectors:TESTPOINT-1mm-NO_TEXT, B.Cu at (159.0, 103.5)
- added J8: D+, RB-SMD-Connectors:TESTPOINT-1mm-NO_TEXT, B.Cu at (159.0, 106.0)
- added J9: GND, RB-SMD-Connectors:TESTPOINT-1mm-NO_TEXT, B.Cu at (153.0, 110.0)
- C1, C10, C12, C2, C3, C4, C5, C6, C7: footprint SMD-DiscreteB:C-0402-1005 -> RB-SMD-DiscreteB:C-0402-1005
- C11: renamed from C8; footprint SMD-DiscreteB:C-0402-1005 -> RB-SMD-DiscreteB:C-0402-1005
- C8: renamed from C9; footprint SMD-DiscreteB:C-0402-1005 -> RB-SMD-DiscreteB:C-0402-1005
- C9: renamed from C11; footprint SMD-DiscreteB:C-0402-1005 -> RB-SMD-DiscreteB:C-0402-1005
- D1: footprint SMD-DiscreteB:LED-0402-1005 -> RB-SMD-DiscreteB:LED-0402-1005
- F1: footprint SMD-DiscreteB:F-0603-1608 -> RB-SMD-DiscreteB:F-0603-1608
- KB1: footprint SMD-Connectors:FPC_0.5mm_22p-MOLEX_52437 -> RB-SMD-Connectors:FPC_0.5mm_22p-MOLEX_52437
- P1: footprint SMD-Connectors:USB-MICRO-10104110-0001LF -> RB-SMD-Connectors:USB-MICRO-10104110-0001LF
- R1: renamed from R3; footprint SMD-DiscreteB:R-0402-1005 -> RB-SMD-DiscreteB:R-0402-1005
- R2: renamed from R1; footprint SMD-DiscreteB:R-0402-1005 -> RB-SMD-DiscreteB:R-0402-1005
- R3: renamed from R2; footprint SMD-DiscreteB:R-0402-1005 -> RB-SMD-DiscreteB:R-0402-1005
- R4, R5: footprint SMD-DiscreteB:R-0402-1005 -> RB-SMD-DiscreteB:R-0402-1005
- SW1: value RST -> RESET; footprint SMD-Switches:ALPS-SKRMAAE010 -> RB-SMD-Switches:ALPS-SKRMAAE010
- U1: footprint SMD-QFN:VQFN-44_ATMEL -> RB-SMD-QFN:VQFN-44_ATMEL
- X1: footprint SMD-XTAL:2.5x2mm -> RB-SMD-XTAL:2.5x2mm
- moved R5 7.07 mm to (161.8, 114.2), turned to 0 degrees
- moved R1 6.40 mm to (161.8, 112.2)
- moved D1 5.83 mm to (161.8, 113.2)
- moved C10 1.27 mm to (169.5, 114.0)
- moved C11 1.27 mm to (164.5, 114.0)
- moved X1 1.27 mm to (167.0, 114.0)
- moved C6 0.56 mm to (168.0, 108.8), turned to 270 degrees
- moved C7 0.56 mm to (168.0, 103.0), turned to 270 degrees
- moved SW1 0.56 mm to (151.8, 113.5)
- moved C12 0.35 mm to (150.8, 109.2)
- moved R4 0.35 mm to (150.8, 110.2)
Connections:
- KB1 pad 4: /COL_10 -> /COL_11
- KB1 pad 5: /COL_11 -> /COL_10
- P1 pad 4: (no net) -> Net-(P1-Pad4)
- U1 pad 20: /COL_10 -> /COL_11
- U1 pad 21: /COL_11 -> /COL_10
- U1 pad 8: (no net) -> /TMP
Routing:
- net /MISO: track 6.12 -> 14.0 mm
- net GND: track 53.1 -> 45.5 mm, vias 12 -> 15
- net /SCK: track 6.79 -> 11.4 mm
- net /RESET: track 14.2 -> 17.3 mm, vias 0 -> 2
- net /LED: track 7.35 -> 5.23 mm
- net +5V: track 55.2 -> 56.7 mm, vias 8 -> 9
- net VBUS: track 3.59 -> 5.09 mm, vias 0 -> 1
- net /D-: track 2.58 -> 3.89 mm, vias 0 -> 1
- net /D+: track 2.58 -> 3.89 mm, vias 0 -> 1
- net /MOSI: track 10.4 -> 9.36 mm
- net Net-(C11-Pad1): track 7.81 -> 8.67 mm
- net /COL_11: track 7.13 -> 7.93 mm
- net /COL_10: track 7.93 -> 7.13 mm
- net Net-(C10-Pad1): track 8.03 -> 8.67 mm
Other:
- board text added: "USB Keyboard v1.22 RasmusB 2018 Psion Series 5/5mx"
- board text removed: "USB Keyboard v1.1 RasmusB 2017 Psion Series 5/5mx"
